Commit message: updated readme

File: install/robot_description/share/robot_description/robot/parts/base/base.xacro (robot description, xacro)
@@ -1 +1,49 @@
-/home/karan/cooperative_marl_ros/src/robot_simulation/robot_description/robot/parts/base/base.xacro
+<?xml version="1.0"?>
+<robot xmlns:xacro="http://ros.org/wiki/xacro">
+  <xacro:include filename="$(find robot_description)/robot/parts/base/base.gazebo"/>
+  <xacro:macro name="base" params="parent robot_name *joint_origin">
+	  <joint name="${robot_name}_base_link_joint" type="fixed">
+	    <xacro:insert_block name="joint_origin"/>
+	    <parent link="${parent}"/>
+	    <child link="${robot_name}_base_link"/>
+	  </joint>
+	<link name="${robot_name}_base_link">
+	  <visual>
+		  <geometry>
+		    <mesh filename="package://robot_description/meshes/DAE/base/base_link_${robot_name}.dae"/>
+		  </geometry>
+	  </visual>
+	  <collision>
+		  <geometry>
+		    <mesh filename="package://robot_description/meshes/STL/base/base_link.stl"/>
+		  </geometry>
+	  </collision>
+	  <inertial>
+		  <origin xyz="0 0 0.32"/>
+		  <mass value="27"/>
+		<inertia ixx="2.2" ixy="0" ixz="0" iyy="9.2" iyz="0" izz="10.6" />
+	  </inertial>
+          <surface>
+            <friction>
+              <ode>
+                <mu>0.8</mu>
+                <mu2>0.8</mu2>
+                <kp>1e15</kp>
+                <kd>1e13</kd>
+              </ode>
+            </friction>
+            <bounce>
+              <restitution_coefficient>0.01</restitution_coefficient>
+              <threshold>10</threshold>
+            </bounce>
+            <contact>
+              <ode>
+                <max_vel>0.01</max_vel>
+                <minDepth>0</minDepth>
+                <contact_surface_layer>0</contact_surface_layer>
+              </ode>
+            </contact>
+          </surface>
+	</link>
+  </xacro:macro>
+</robot>

File: install/robot_description/share/robot_description/robot/parts/knuckle/knuckle.xacro (robot description, xacro)
@@ -1 +1,50 @@
-/home/karan/cooperative_marl_ros/src/robot_simulation/robot_description/robot/parts/knuckle/knuckle.xacro
+<?xml version="1.0"?>
+<robot xmlns:xacro="http://ros.org/wiki/xacro">
+  <xacro:include filename="$(find robot_description)/robot/parts/knuckle/knuckle.gazebo"/>
+  <xacro:macro name="knuckle" params="prefix parent *joint_origin *joint_axis">
+	<joint name="${prefix}_knuckle_joint" type="revolute">
+	  <xacro:insert_block name="joint_origin"/>
+	  <parent link="${parent}"/>
+	  <child link="${prefix}_knuckle_link"/>
+          <limit effort="200" velocity="3" lower="-1.51" upper = "1.51"/>
+          <dynamics damping="0.005" friction="0.1"/>
+	  <xacro:insert_block name="joint_axis"/>
+	</joint>
+	<link name="${prefix}_knuckle_link">
+	  <visual>
+		  <geometry>
+		    <mesh filename="package://robot_description/meshes/STL/knuckle/knuckle.stl"/>
+		  </geometry>
+	  </visual>
+	  <collision>
+		  <geometry>
+		    <mesh filename="package://robot_description/meshes/STL/knuckle/knuckle.stl"/>
+		  </geometry>
+	  </collision>
+    <inertial>
+		<origin xyz="0.0 -0.011 -0.0"/>
+		<mass value="0.25"/>
+		<inertia ixx="0.00031" ixy="0" ixz="0" iyy="0.0005" iyz="0" izz="0.00031"/>
+	  </inertial>
+          <surface>
+            <friction>
+              <ode>
+                <mu1>1.2</mu1>
+                <mu2>1.2</mu2>
+                <kp>1e15</kp>
+                <kd>1e13</kd>
+              </ode>
+            </friction>
+            <bounce>
+              <restitution_coefficient>0.01</restitution_coefficient>
+              <threshold>0</threshold>
+            </bounce>
+            <contact>
+              <ode>
+                <max_vel>10</max_vel>
+              </ode>
+            </contact>
+          </surface>
+	</link>
+  </xacro:macro>
+</robot>

File: install/robot_description/share/robot_description/robot/parts/wheel/wheel.xacro (robot description, xacro)
@@ -1 +1,49 @@
-/home/karan/cooperative_marl_ros/src/robot_simulation/robot_description/robot/parts/wheel/wheel.xacro
+<?xml version="1.0"?>
+<robot xmlns:xacro="http://ros.org/wiki/xacro">
+  <xacro:include filename="$(find robot_description)/robot/parts/wheel/wheel.gazebo"/>
+  <xacro:macro name="wheel" params="prefix parent *joint_origin *joint_axis">
+	<joint name="${prefix}_wheel_joint" type="continuous">
+	  <xacro:insert_block name="joint_origin"/>
+	  <parent link="${parent}"/>
+	  <child link="${prefix}_wheel_link"/>
+          <limit effort="100" velocity="100"/>
+	  <xacro:insert_block name="joint_axis"/>
+	</joint>
+	<link name="${prefix}_wheel_link">
+	  <visual>
+		  <geometry>
+		    <mesh filename="package://robot_description/meshes/DAE/wheel/wheel.dae"/>
+		  </geometry>
+	  </visual>
+	  <collision>
+		  <geometry>
+		    <mesh filename="package://robot_description/meshes/STL/wheel/wheel.stl"/>
+		  </geometry>
+	  </collision>
+	  <inertial>
+		<origin xyz="0.0 0.0 0.0"/>
+		<mass value="1.0"/>
+		<inertia ixx="0.222" ixy="0" ixz="0" iyy="0.395" iyz="0" izz="0.222"/>
+	  </inertial>
+          <surface>
+            <friction>
+              <ode>
+                <mu1>1.2</mu1>
+                <mu2>1.2</mu2>
+                <kp>1e15</kp>
+                <kd>1e13</kd>
+              </ode>
+            </friction>
+            <bounce>
+              <restitution_coefficient>0.01</restitution_coefficient>
+              <threshold>0</threshold>
+            </bounce>
+            <contact>
+              <ode>
+                <max_vel>10</max_vel>
+              </ode>
+            </contact>
+          </surface>
+	</link>
+  </xacro:macro>
+</robot>

File: install/robot_description/share/robot_description/robot/robot.xacro (robot description, xacro)
@@ -1 +1,53 @@
-/home/karan/cooperative_marl_ros/src/robot_simulation/robot_description/robot/robot.xacro
+<?xml version="1.0"?>
+<robot name="omni_robot" xmlns:xacro="http://ros.org/wiki/xacro">
+  <xacro:include filename="$(find robot_description)/robot/parts/base/base.xacro"/>
+  <xacro:include filename="$(find robot_description)/robot/parts/wheel/wheel.xacro"/>
+  <xacro:include filename="$(find robot_description)/robot/parts/knuckle/knuckle.xacro"/>
+  <xacro:include filename="$(find robot_description)/robot/robot_control_gazebo.xacro"/>
+  <xacro:property name="PI" value="3.14159274"/>
+  <xacro:arg name="robot_name" default="robot_1"/>
+  <!-- =============== Link & Joint =============== -->
+  <!-- Base -->
+  <link name="$(arg robot_name)_base_footprint"/>
+  <xacro:base robot_name="$(arg robot_name)" parent="$(arg robot_name)_base_footprint">
+    <origin xyz="0 0 0" rpy="0 0 0" />
+  </xacro:base>
+  <!-- Suspension -->
+  <!-- Front Right Sus -->
+  <xacro:knuckle prefix="$(arg robot_name)_front_right" parent="$(arg robot_name)_base_link">
+	<origin xyz="0.9 -0.55 0.05" rpy="0 0 ${PI}"/>
+	<axis xyz="0 0 1"/>
+  </xacro:knuckle>
+  <!-- Front Left Sus -->
+  <xacro:knuckle prefix="$(arg robot_name)_front_left" parent="$(arg robot_name)_base_link">
+	<origin xyz="0.9 0.55 0.05" rpy="0 0 0"/>
+	<axis xyz="0 0 1"/>
+  </xacro:knuckle>
+  <!-- Wheels -->
+  <xacro:wheel prefix="$(arg robot_name)_fr" parent="$(arg robot_name)_front_right_knuckle_link">
+	  <origin xyz="0.0 0.0 0.0" rpy="0 0 0"/>
+	  <axis xyz="0 -1 0"/>
+  </xacro:wheel>
+  <xacro:wheel prefix="$(arg robot_name)_fl" parent="$(arg robot_name)_front_left_knuckle_link">
+	<origin xyz="0.0 0.0 0.0" rpy="0 0 0"/>
+	<axis xyz="0 1 0"/>
+  </xacro:wheel>
+  <xacro:wheel prefix="$(arg robot_name)_rl" parent="$(arg robot_name)_base_link">
+	<origin xyz="-0.9 0.55 0.05" rpy="0 0 0"/>
+	<axis xyz="0 1 0"/>
+  </xacro:wheel>
+  <xacro:wheel prefix="$(arg robot_name)_rr" parent="$(arg robot_name)_base_link">
+	<origin xyz="-0.9 -0.55 0.05" rpy="0 0 ${PI}"/>
+	<axis xyz="0 -1 0"/>
+  </xacro:wheel>
+  <!-- =============== Gazebo =============== -->
+  <!-- Controllers -->
+  <xacro:robot_gazebo_systems robot_name="$(arg robot_name)"/>
+  <!-- Base -->
+  <xacro:base_gazebo_v0 robot_name="$(arg robot_name)"/>
+  <!-- Wheels -->
+  <xacro:wheel_gazebo_v0 prefix="$(arg robot_name)_fr"/>
+  <xacro:wheel_gazebo_v0 prefix="$(arg robot_name)_fl"/>
+  <xacro:wheel_gazebo_v0 prefix="$(arg robot_name)_rl"/>
+  <xacro:wheel_gazebo_v0 prefix="$(arg robot_name)_rr"/>
+</robot>

File: install/robot_description/share/robot_description/robot/robot_control_gazebo.xacro (robot description, xacro)
@@ -1 +1,59 @@
-/home/karan/cooperative_marl_ros/src/robot_simulation/robot_description/robot/robot_control_gazebo.xacro
+<?xml version="1.0" ?>
+<robot xmlns:xacro="http://www.ros.org/wiki/xacro">
+<xacro:macro  name="robot_gazebo_systems" params="robot_name">
+  <ros2_control name="${robot_name}_GazeboSystem" type="system">
+    <hardware>
+      <plugin>gazebo_ros2_control/GazeboSystem</plugin>
+    </hardware>
+    <joint name="${robot_name}_front_right_knuckle_joint">
+      <command_interface name="position">
+        <param name="min">-3.14</param>
+        <param name="max">3.14</param>
+      </command_interface>
+      <state_interface name="position"/>
+    </joint>
+    <joint name="${robot_name}_front_left_knuckle_joint">
+      <command_interface name="position">
+        <param name="min">-3.14</param>
+        <param name="max">3.14</param>
+      </command_interface>
+      <state_interface name="position"/>
+    </joint>
+    <joint name="${robot_name}_rl_wheel_joint">
+      <command_interface name="velocity">
+        <param name="min">-3.14</param>
+        <param name="max">3.14</param>
+      </command_interface>
+      <state_interface name="velocity"/>
+    </joint>
+    <joint name="${robot_name}_rr_wheel_joint">
+      <command_interface name="velocity">
+        <param name="min">-3.14</param>
+        <param name="max">3.14</param>
+      </command_interface>
+      <state_interface name="velocity"/>
+    </joint>
+  </ros2_control>
+  <gazebo>
+    <plugin name="${robot_name}_joint_state" filename="libgazebo_ros_joint_state_publisher.so">
+      <ros>
+        <namespace>${robot_name}</namespace>
+      </ros>
+      <update_rate>20</update_rate>
+      <joint_name>${robot_name}_fr_wheel_joint</joint_name>
+      <joint_name>${robot_name}_fl_wheel_joint</joint_name>
+      <joint_name>${robot_name}_rl_wheel_joint</joint_name>
+      <joint_name>${robot_name}_rr_wheel_joint</joint_name>
+      <joint_name>${robot_name}_front_right_knuckle_joint</joint_name>
+      <joint_name>${robot_name}_front_left_knuckle_joint</joint_name>
+    </plugin>
+    <plugin filename="libgazebo_ros2_control.so" name="${robot_name}_gazebo_ros2_control">
+        <ros>
+          <namespace>${robot_name}</namespace>
+        </ros>
+        <parameters>$(find robot_description)/config/${robot_name}_controller.yaml</parameters>
+        <robot_param_node>/${robot_name}_robot_state_publisher</robot_param_node>
+    </plugin>
+  </gazebo>
+</xacro:macro >
+</robot>
